File: Hardware/LEDsignPCB.kicad_sch (KiCad schematic)
At the start: 46 parts, among them SW1 SW_Push, SW2 SW_Push, U1 ESP32-S3-WROOM-1, U2 AMS1117-3.3, U3 SN74HCT125N, U4 TPS54332DDA

Commit message: finished rough schematic!
Parts:
- removed C6: 1u, symbol Device:C
- removed R10: 100k, symbol Device:R
- removed R11, R9: R, symbol Device:R
- removed R8: 6.8k, symbol Device:R
- removed U?: CH224K, Package_SO:SSOP-10-1EP_3.9x4.9mm_P1mm_EP2.1x3.3mm, symbol Interface_USB:CH224K
- added C18, C26: 10u, symbol Device:C
- added C19, C22, C24, C25, C28, C31, C32: 100n, symbol Device:C_Small
- added C20, C21: 1000u, symbol Device:C
- added C23, C29, C30: 1u, symbol Device:C
- added C27: .1u, symbol Device:C_Small
- added J1, J2: Conn_01x03, symbol Connector_Generic:Conn_01x03
- added J3, J4: Conn_01x04, symbol Connector_Generic:Conn_01x04
- added Q1: AO3401A, Package_TO_SOT_SMD:SOT-23, symbol Transistor_FET:AO3401A
- added R16, R17: 330, symbol Device:R_Small
- added R18, R21, R22, R24, R25, R26, R28, R29, R30, R31: 100k, symbol Device:R
- added R19, R20: 4.7k, symbol Device:R_Small
- added R23: 22k, symbol Device:R
- added R27: R_Small, symbol Device:R_Small
- added U5: RT9193-33GB, SOT-23-5_RIT, symbol LED Sign:RT9193-33GB
- added U6: STUSB4500QTR, Package_DFN_QFN:QFN-24-1EP_4x4mm_P0.5mm_EP2.7x2.7mm, symbol Interface_USB:STUSB4500QTR
- F1: value Polyfuse -> Polyfuse (3A)
Connections:
- net +3V3: now also C18.1, C19.1, C26.2, J3.1 (Pin_1), J4.1 (Pin_1), R19.1, R20.1, R28.1, R30.2, U5.1 (VIN), U5.3 (EN)
- net +5V: now also U3.14 (VCC), C20.1, C21.1, C22.1, J1.1 (Pin_1), J2.1 (Pin_1)
- net +9V: now also Q1.3 (D)
- net CC1: now also U6.1 (CC1DB), U6.2 (CC1)
- net CC2: now also U6.4 (CC2), U6.5 (CC2DB)
- net GND: now also MK2.2 (LR), MK2.3 (GND), U3.1 (*1OE), U3.4 (*2OE), U3.7 (GND), C18.2, C19.2, C20.2, C21.2, C22.2, C23.2, C24.2, C25.2, C27.1, C28.2, C29.1, C30.1, C31.2, C32.2, J1.3 (Pin_3), J2.3 (Pin_3), J3.4 (Pin_4), J4.4 (Pin_4), R18.2, R24.1, R27.2, U5.2 (GND), U6.10 (GND), U6.12 (ADDR0), U6.13 (ADDR1), U6.22 (VSYS), U6.25 (GND)
- net LED1: now also R16.2
- net LED2: now also R17.2
- net RESET: now also U1.18 (IO10), C32.1, R24.2, U6.6 (RESET)
- net SD: now reaches U1.10 (IO17)
- net SD: now also MK2.6 (SD), R18.1
- net SDA: now reaches U1.12 (IO8)
- net SDA: now also J4.2 (Pin_2), R19.2, U6.8 (SDA)
- net SCL: now reaches U1.17 (IO9)
- net SCL: now also J4.3 (Pin_3), R20.2, U6.7 (SCL)
- net at C5.2, C7.2, C8.2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: now also C26.1
- net RX: now reaches U1.36 (RXD0)
- net RX: now also J3.3 (Pin_3)
- net TX: now reaches U1.37 (TXD0)
- net TX: now also J3.2 (Pin_2)
- net ATTACH: now reaches U1.6 (IO6)
- net ATTACH: now also R26.1, U6.11 (ATTACH)
- net FAULT: now reaches U1.7 (IO7)
- net FAULT: now also R25.1, U6.15 (GPIO)
- net SCK: now reaches U1.8 (IO15)
- net SCK: now also MK2.4 (SCK)
- net WS: now reaches U1.9 (IO16)
- net WS: now also MK2.1 (WS)
- net at D2.1 (K): now also C28.1, U6.24 (VDD)
- net 3V3_MIC: now reaches MK2.5 (VDD)
- net 3V3_MIC: now also C23.1, C24.1, C27.2, U5.5 (VOUT)
- net at U3.2 (1A): now also R16.1
- net DATA1: now reaches U3.3 (1Y)
- net DATA1: now also U3.6 (2Y), J1.2 (Pin_2)
- net at U3.5 (2A): now also R17.1
- net PG renamed EN
- net EN: now also R29.1, U6.20 (POWER_OK2)
- net VBUS_IN renamed VBUS
- net VBUS: now also Q1.2 (S), R21.1, R22.2, R23.1, R25.2, R26.2, R29.2, R31.2
- new net: C31.1, Q1.1 (G), R22.1, R23.2, U6.16 (VBUS_EN_SNK)
- new net: R21.2, U6.18 (VBUS_VS_DISCH)
- new net: C29.2, U6.21 (VREG_1V2)
- new net: R30.1, U6.14 (POWER_OK3)
- new net: R28.2, U6.17 (A_B_SIDE)
- new net: C30.2, U6.23 (VREG_2V7)
- new net: R27.1, U6.9 (DISCH)
- new net: C25.1, U5.4 (BP)
- new net ALERT: R31.1, U6.19 (ALERT)
- new net DATA2: J2.2 (Pin_2)
- no-connect marks 12 -> 34
Other:
- note added: "I2C expansion (light sensor?)"
- note added: "UART recovery header"
- note added: "active high, maybe route to GPIO"
- note added: "both ceramic"
- note added: "bottom ported mic add hole beneath mic slightly larger than port diameter in footprint dont use via since solder will stick"
- note added: "bottom ported mic!!!"
- note added: "ceramic x7r"
- note added: "damp gate oscillation and slow turn on, prevent inrush current spike"
- note added: "default I2C address: 0x28"
- note added: "ensures gate voltage tracks source voltage"
- note added: "keep mic far away from sw node and inductor"
- note added: "no vias"
- note added: "place close to pin filters noise on internal reference voltage"
- note added: "pulls gate high"
- note added: "single layer"
- note removed: "as close to pin as possible"
- moved on the sheet: C1, C4, C5, C7, C8, D1, D2, F1, J?, MK2, R1, R2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

Commit message: some organization, switch to desktop
Parts:
- added J5: USB_C_Receptacle_USB2.0_14P, symbol Connector:USB_C_Receptacle_USB2.0_14P
Connections:
- net CC1: now also J5.A5 (CC1)
- net CC2: now also J5.B5 (CC2)
- net VBUS: now also J5.A4 (VBUS), J5.A9 (VBUS), J5.B4 (VBUS), J5.B9 (VBUS)
- new net: J5.A1 (GND), J5.A12 (GND), J5.B1 (GND), J5.B12 (GND)
- new net Power Protection/D+: J5.A6 (D+), J5.B6 (D+)
- new net Power Protection/D-: J5.A7 (D-), J5.B7 (D-)
Other:
- added sheet PD Negotiation (pdnegotiation.kicad_sch)
- added sheet Power Protection (powerprotection.kicad_sch)

Commit message: made subsheets and cleaned up, still need to make schematic even better
Parts:
- removed C1: 100nF, symbol Device:C_Small
- removed C10, C13, C14, C19, C2, C22, C24, C25, C28, C31, C32, C4, C5, C7, C8: 100n, symbol Device:C_Small
- removed C11, C12: 47u, symbol Device:C
- removed C15: 8.2n, symbol Device:C
- removed C16: 20p, symbol Device:C_Small
- removed C17: 1n, symbol Device:C_Small
- removed C18, C26, C3: 10u, symbol Device:C
- removed C23, C29, C30: 1u, symbol Device:C
- removed C27: .1u, symbol Device:C_Small
- removed C9: 22u, symbol Device:C
- removed D1: PRTR5V0U2X, Package_TO_SOT_SMD:SOT-143, symbol Power_Protection:PRTR5V0U2X
- removed D2: D_Schottky, symbol Device:D_Schottky
- removed D3: SS34, Diode_SMD:D_SMA, symbol Diode:SS34
- removed F1: Polyfuse (3A), Fuse:Fuse_1206_3216Metric_Pad1.42x1.75mm_HandSolder, symbol Device:Polyfuse
- removed J?: USB_C_Receptacle, Connector_USB:USB_C_Receptacle_GCT_USB4085, symbol Connector:USB_C_Receptacle
- removed L1: 2.5u, symbol Device:L
- removed MK2: ICS-43434, Sensor_Audio:InvenSense_ICS-43434-6_3.5x2.65mm, symbol Sensor_Audio:ICS-43434
- removed Q1: AO3401A, Package_TO_SOT_SMD:SOT-23, symbol Transistor_FET:AO3401A
- removed R1, R2: 5.1k, symbol Device:R_Small
- removed R12, R18, R21, R22, R24, R25, R26, R28, R29, R30, R31: 100k, symbol Device:R
- removed R13: 10.2k, symbol Device:R
- removed R14: 1.96k, symbol Device:R
- removed R15: 69.8k, symbol Device:R
- removed R16, R17: 330, symbol Device:R_Small
- removed R19, R20: 4.7k, symbol Device:R_Small
- removed R23: 22k, symbol Device:R
- removed R27: R_Small, symbol Device:R_Small
- removed R3, R4, R5, R6, R7: 10k, symbol Device:R_Small
- removed SW1, SW2: SW_Push, symbol Switch:SW_Push
- removed U1: ESP32-S3-WROOM-1, RF_Module:ESP32-S3-WROOM-1, symbol RF_Module:ESP32-S3-WROOM-1
- removed U2: AMS1117-3.3, Package_TO_SOT_SMD:SOT-223-3_TabPin2, symbol Regulator_Linear:AMS1117-3.3
- removed U3: SN74HCT125N, N14, symbol LED Sign:SN74HCT125N
- removed U4: TPS54332DDA, DDA8_3X2P13, symbol LED Sign:TPS54332DDA
- removed U5: RT9193-33GB, SOT-23-5_RIT, symbol LED Sign:RT9193-33GB
- removed U6: STUSB4500QTR, Package_DFN_QFN:QFN-24-1EP_4x4mm_P0.5mm_EP2.7x2.7mm, symbol Interface_USB:STUSB4500QTR
- added C55: 10u, symbol Device:C
- added C56, C57, C58, C60, C62: 100n, symbol Device:C_Small
- added C59: 100nF, symbol Device:C_Small
- added C61: 1u, symbol Device:C_Small
- added R39, R40: 5.1k, symbol Device:R_Small
- added R42, R43: 4.7k, symbol Device:R_Small
- added R44, R45: 10k, symbol Device:R_Small
- added R57, R58: 22, symbol Device:R_Small
- added R59: 499, symbol Device:R_Small
- added SW5, SW6: SW_Push, symbol Switch:SW_Push
- added U12: ESP32-S3-WROOM-1, RF_Module:ESP32-S3-WROOM-1, symbol RF_Module:ESP32-S3-WROOM-1
Connections:
- net +3V3: now also C55.2, C56.1, C57.1, C58.1, R42.1, R43.1, R44.1, R45.1
- net ALERT: now also U12.35 (IO42)
- net ATTACH: now also U12.33 (IO40)
- net CC1: now also R39.1
- net CC2: now also R40.1
- net EN: now also C61.1, R44.2, SW5.2, U12.3 (EN)
- net FAULT: now also U12.34 (IO41)
- net GND: now also J5.A1 (GND), J5.A12 (GND), J5.B1 (GND), J5.B12 (GND), C59.2, C60.2, C61.2, C62.2, R39.2, R40.2, SW5.1, SW6.1, U12.1 (GND), U12.40 (GND), U12.41 (GND)
- net LED1: now also U12.31 (IO38)
- net LED2: now also U12.32 (IO39)
- net RESET: now also U12.18 (IO10)
- net RX: now also U12.36 (RXD0)
- net SCK: now also U12.8 (IO15)
- net SCL: now also R43.2, U12.17 (IO9)
- net SD: now also U12.10 (IO17)
- net SDA: now also R42.2, U12.12 (IO8)
- net TX: now also R59.1, U12.37 (TXD0); no longer J3.2 (Pin_2)
- net WS: now also U12.9 (IO16)
- net at J5.SH (SHIELD): now also C59.1
- new net: C55.1, C56.2, C57.2, C58.2, U12.2 (3V3)
- new net: R45.2, SW6.2, U12.27 (IO0)
- new net: R57.2, U12.13 (USB_D-)
- new net: R58.2, U12.14 (USB_D+)
- new net: J3.2 (Pin_2), R59.2
- new net D+: C60.1, R58.1
- new net D-: C62.1, R57.1
- no-connect marks 34 -> 20
Other:
- added sheet 3.3V Filter (filter.kicad_sch)
- added sheet 3.3V-5V Level Shifter (levelshifter.kicad_sch)
- added sheet 5V-3.3V LDO (LDO.kicad_sch)
- added sheet 9V-5V Buck Converter (buckconverter.kicad_sch)
- added sheet Microphone (microphone.kicad_sch)
- sheet PD Negotiation ports: added ALERT, ATTACH, CC1, CC2, EN, FAULT, PD_IN, PD_OUT, RESET, SCL, SDA; removed none
- note added: "I2C Pull-ups"
- note removed: "Vout = Vref × (1 + Rfbt/Rfbb) Vout = 0.8 × (1 + 10.2k/1.96k) Vout = 0.8 × (1 + 5.204) Vout = 0.8 × 6.204 = 4.96V ≈ 5V ✅ use E96 resistors"
- note removed: "active high, maybe route to GPIO"
- note removed: "both ceramic"
- note removed: "bottom ported mic add hole beneath mic slightly larger than port diameter in footprint dont use via since solder will stick"
- note removed: "bottom ported mic!!!"
- note removed: "ceramic"
- note removed: "ceramic HF noise"
- note removed: "ceramic X7R"
- note removed: "ceramic X7R 16V+ rated"
- note removed: "ceramic x7r"
- note removed: "choose X7R voltage rating at least 2x 3x higher"
- note removed: "damp gate oscillation and slow turn on, prevent inrush current spike"
- note removed: "default I2C address: 0x28"
- note removed: "electrolytic bulk stability"
- note removed: "ensures gate voltage tracks source voltage"
- note removed: "keep mic far away from sw node and inductor"
- note removed: "no vias"
- note removed: "physically place close to receptacle"
- note removed: "place close to SW pin as possible short trace to GND 450mV, 3A Schottky diode"
- note removed: "place close to VIN pin"
- note removed: "place close to pin filters noise on internal reference voltage"
- note removed: "pulls gate high"
- note removed: "saturation current rating >= 4.5A use shielded inductor"
- note removed: "single layer"
- note removed: "use at least 10V rated caps"
- moved on the sheet: C20, C21, J1, J2, J3, J4, J5
