File: Hardware/LEDsignPCB.kicad_sch (KiCad schematic)
At the start: 0 parts

Commit message: polished up schematic
Other:
- note added: "- Designed for PD source with 9V or higher profile - Use 5V addressable strips (WS2812B) - PD controller must initially be programmed through NVM to accept profiles greater than 5V - Reset hardware: press RESET button - Entering bootloader: hold BOOT (GPIO0 is strapping), press RESET, release BOOT. - Run firmware: press RESET"
- note removed: "- Designed for any PD charger with 9V or higher profile - Use 5V addressable strips - must initially NVM program PD controllerto accept profiles >5V - RESET button to reset hardware - Entering flash mode: hold BOOT, press and release RESET, then release BOOT. - Entering run mode: press RESET (BOOT is already pulled high)"
- company: (none) -> Jennifer Li
- title: (none) -> WS2812B Driver PCB
Changed lines of the file:
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@@
 	(generator_version "10.0")
 	(paper "A4")
+	(title_block
+		(title "WS2812B Driver PCB")
+		(date "7/2026")
+		(rev "RevA")
+		(company "Jennifer Li")
+	)
 	(rectangle
 		(start 177.8 127.762)
@@
 		)
 	)
-	(text "- Designed for any PD charger with 9V or higher profile\n- Use 5V addressable strips\n- must initially NVM program PD controllerto accept profiles >5V\n- RESET button to reset hardware\n- Entering flash mode: hold BOOT, press and release RESET, then\nrelease BOOT.\n- Entering run mode: press RESET (BOOT is already pulled high)"
+	(text "- Designed for PD source with 9V or higher profile\n- Use 5V addressable strips (WS2812B)\n- PD controller must initially be programmed through NVM to \naccept profiles greater than 5V\n- Reset hardware: press RESET button\n- Entering bootloader: hold BOOT (GPIO0 is strapping), \npress RESET, release BOOT.\n- Run firmware: press RESET"
 		(exclude_from_sim no)
 		(at 180.086 147.066 0)
@@
 		(dnp no)
 		(fields_autoplaced yes)
-		(property "Reference" "#PWR022"
+		(property "Reference" "#PWR01"
 			(at 27.94 64.77 0)
 			(hide yes)
@@
 			(project "LEDsignPCB"
 				(path "/bd70e714-05b6-457c-88d3-c29e19a48f7d"
-					(reference "#PWR022")
+					(reference "#PWR01")
 					(unit 1)
 				)
@@
 		(dnp no)
 		(fields_autoplaced yes)
-		(property "Reference" "#PWR015"
+		(property "Reference" "#PWR02"
 			(at 69.85 175.26 0)
 			(hide yes)
@@
 			(project "LEDsignPCB"
 				(path "/bd70e714-05b6-457c-88d3-c29e19a48f7d"
-					(reference "#PWR015")
+					(reference "#PWR02")
 					(unit 1)
 				)
@@
 		(dnp no)
 		(fields_autoplaced yes)
-		(property "Reference" "#PWR024"
+		(property "Reference" "#PWR04"
 			(at 238.76 124.46 0)
 			(hide yes)
@@
 			(project "LEDsignPCB"
 				(path "/bd70e714-05b6-457c-88d3-c29e19a48f7d"
-					(reference "#PWR024")
+					(reference "#PWR04")
 					(unit 1)
 				)
@@
 		(dnp no)
 		(fields_autoplaced yes)
-		(property "Reference" "#PWR023"
+		(property "Reference" "#PWR03"
 			(at 90.17 72.39 0)
 			(hide yes)
@@
 			(project "LEDsignPCB"
 				(path "/bd70e714-05b6-457c-88d3-c29e19a48f7d"
-					(reference "#PWR023")
+					(reference "#PWR03")
 					(unit 1)
 				)

Commit message: final touches to sch, switch out microphone
Other:
- sheet LEDs and Audio (page 5) ports: added BCLK, MIC_DATA; removed SCK, SD
Changed lines of the file:
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@@
-			)
-		)
-		(pin "SCK" input
-			(at 203.2 110.49 180)
-			(effects
-				(font
-					(size 1.27 1.27)
-				)
-				(justify left)
-			)
-		)
-		(pin "SD" input
-			(at 203.2 114.3 180)
-			(effects
-				(font
-					(size 1.27 1.27)
-				)
-				(justify left)
 			)
 		)
@@
 			)
 		)
+		(pin "BCLK" input
+			(at 203.2 110.49 180)
+			(effects
+				(font
+					(size 1.27 1.27)
+				)
+				(justify left)
+			)
+		)
+		(pin "MIC_DATA" input
+			(at 203.2 114.3 180)
+			(effects
+				(font
+					(size 1.27 1.27)
+				)
+				(justify left)
+			)
+		)
