File: Hardware/InputProtection.kicad_sch (KiCad schematic)
At the start: 13 parts, among them J6 USB_C_Receptacle_USB2.0_14P

Commit message: switch to desktop
Parts:
- added TP17: GND, symbol Connector:TestPoint
- D8: value LED_Small -> VBUS
- D9: value LED_Small -> VBUS_PP
- TP1: value TestPoint -> VBUS
- TP2: value TestPoint -> VBUS_PP
Connections:
- net GND: now also TP17.1
Other:
- moved on the sheet: TP1, TP2

Commit message: polished up schematic
Parts:
- removed TP17: GND, symbol Connector:TestPoint
- renumbered C63 to C1, D8 to D1, D9 to D2, D4 to D3, D5 to D4, F2 to F1, J6 to J1, R41 to R1, R60 to R2, R14 to R4
Other:
- note added: "1. keep TVS and receptacle tight 2. avoid traces parallel to signal path 3. minimize conductive loops (PWR & GND) 4. minimize ground return path length 5. avoid sharing ground return paths 6. use ground planes and ground vias"
- note removed: "1. keep tvs and receptacle very tight 2. avoid traces parallel to signal path 3. minimize conductive loops (PWR & GND) 4. minimize ground return path length 5. avoid sharing ground return paths 6. use ground planes or ground vias"
- company: (none) -> Jennifer Li
- title: (none) -> USBC Receptacle + Protection Circuitry
- moved on the sheet: TP1, TP2
