File: Hardware/InputProtection.kicad_sch (KiCad schematic)
At the start: 13 parts, among them J1 USB_C_Receptacle_USB2.0_14P

Commit message: switch to macbook
Parts:
- C1: value 100nF -> 100n; footprint (none) -> Capacitor_SMD:C_0603_1608Metric_Pad1.08x0.95mm_HandSolder; P/N (none) -> GRM188R72A104KA35D
- D1: footprint (none) -> LED_SMD:LED_0805_2012Metric_Pad1.15x1.40mm_HandSolder; P/N (none) -> LTST-C170GKT
Changed lines of the file:
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@@
 			)
 		)
-		(property "Footprint" ""
+		(property "Footprint" "LED_SMD:LED_0805_2012Metric_Pad1.15x1.40mm_HandSolder"
 			(at 115.57 36.83 90)
 			(hide yes)
@@
 		)
 		(property " LCSC P/N" ""
+			(at 115.57 36.83 90)
+			(hide yes)
+			(show_name no)
+			(do_not_autoplace no)
+			(effects
+				(font
+					(size 1.27 1.27)
+				)
+			)
+		)
+		(property "P/N" "LTST-C170GKT"
 			(at 115.57 36.83 90)
 			(hide yes)
@@
 			)
 		)
-		(property "Value" "100nF"
+		(property "Value" "100n"
 			(at 34.036 85.852 0)
 			(show_name no)
@@
 			)
 		)
-		(property "Footprint" ""
+		(property "Footprint" "Capacitor_SMD:C_0603_1608Metric_Pad1.08x0.95mm_HandSolder"
 			(at 40.64 83.82 0)
 			(hide yes)
@@
 			)
 		)
-		(property "P/N" ""
+		(property "P/N" "GRM188R72A104KA35D"
 			(at 40.64 83.82 0)
 			(hide yes)

Commit message: final touches to sch, switch out microphone
Parts:
- D1: value VBUS -> VBUS_LED
- D2: value VBUS_PP -> VBUS_PP_LED; footprint (none) -> LED_SMD:LED_0805_2012Metric_Pad1.15x1.40mm_HandSolder; P/N (none) -> LTST-C170GKT
- D3: P/N (none) -> PRTR5V0U2X,215
- J1: footprint (none) -> Connector_USB:USB_C_Receptacle_GCT_USB4105-xx-A_16P_TopMnt_Horizontal; P/N (none) -> USB4105-GF-A-060
- R1, R2: footprint (none) -> Resistor_SMD:R_0603_1608Metric_Pad0.98x0.95mm_HandSolder
- R3, R4: value R_Small -> R
- TP1: value VBUS -> VBUS_TP; footprint (none) -> TestPoint:TestPoint_Keystone_5000-5004_Miniature
- TP2: value VBUS_PP -> VBUS_PP_TP; footprint (none) -> TestPoint:TestPoint_Keystone_5000-5004_Miniature
Changed lines of the file:
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@@
 			)
 		)
-		(property "Value" "R_Small"
+		(property "Value" "R"
 			(at 134.62 33.0199 0)
 			(show_name no)
@@
 			)
 		)
-		(property "Footprint" ""
+		(property "Footprint" "Resistor_SMD:R_0603_1608Metric_Pad0.98x0.95mm_HandSolder"
 			(at 72.39 48.26 0)
 			(hide yes)
@@
 			)
 		)
-		(property "P/N" ""
+		(property "P/N" "PRTR5V0U2X,215"
 			(at 146.05 74.93 0)
 			(hide yes)
@@
 			)
 		)
-		(property "Value" "R_Small"
+		(property "Value" "R"
 			(at 118.11 33.0199 0)
 			(show_name no)
@@
 			)
 		)
-		(property "Footprint" ""
+		(property "Footprint" "Connector_USB:USB_C_Receptacle_GCT_USB4105-xx-A_16P_TopMnt_Horizontal"
 			(at 52.07 58.42 0)
 			(hide yes)
@@
 			)
 		)
+		(property "P/N" "USB4105-GF-A-060"
+			(at 48.26 58.42 0)
+			(hide yes)
+			(show_name no)
+			(do_not_autoplace no)
+			(effects
+				(font
+					(size 1.27 1.27)
+				)
+			)
+		)
 		(pin "A1"
 		)
@@
 			)
 		)
-		(property "Value" "VBUS"
+		(property "Value" "VBUS_LED"
 			(at 117.348 38.608 90)
 			(show_name no)
@@
 			)
 		)
-		(property "Value" "VBUS_PP"
+		(property "Value" "VBUS_PP_LED"
 			(at 134.62 38.354 90)
 			(show_name no)
@@
 			)
 		)
-		(property "Footprint" ""
+		(property "Footprint" "LED_SMD:LED_0805_2012Metric_Pad1.15x1.40mm_HandSolder"
 			(at 132.08 36.83 90)
 			(hide yes)
@@
 			)
 		)
+		(property "P/N" "LTST-C170GKT"
+			(at 132.08 36.83 90)
+			(hide yes)
+			(show_name no)
+			(do_not_autoplace no)
+			(effects
+				(font
+					(size 1.27 1.27)
+				)
+			)
+		)
 		(pin "2"
 		)
@@
 			)
 		)
-		(property "Value" "VBUS_PP"
+		(property "Value" "VBUS_PP_TP"
 			(at 173.99 32.2579 0)
 			(show_name no)
@@
 			)
 		)
-		(property "Footprint" ""
+		(property "Footprint" "TestPoint:TestPoint_Keystone_5000-5004_Miniature"
 			(at 176.53 34.29 0)
 			(hide yes)
@@
 			)
 		)
-		(property "Value" "VBUS"
+		(property "Value" "VBUS_TP"
 			(at 160.02 32.2579 0)
 			(show_name no)
@@
 			)
 		)
-		(property "Footprint" ""
+		(property "Footprint" "TestPoint:TestPoint_Keystone_5000-5004_Miniature"
 			(at 162.56 34.29 0)
 			(hide yes)
@@
 			)
 		)
-		(property "Footprint" ""
+		(property "Footprint" "Resistor_SMD:R_0603_1608Metric_Pad0.98x0.95mm_HandSolder"
 			(at 72.39 50.8 0)
 			(hide yes)
