File: Hardware/MCU.kicad_sch (KiCad schematic)
At the start: 31 parts, among them J10 Conn_01x04, J9 Conn_01x04, SW7 SW_Push, SW8 SW_Push, U16 ESP32-S3-WROOM-1

Commit message: switch to desktop
Parts:
- D11: value LED_Small -> RX
- D12: value LED_Small -> RESET
- D13: value LED_Small -> BOOT
- D7: value LED_Small -> TX
- R10: value R_Small -> RESET
- R19: value R_Small -> BOOT
- R8: value R_Small -> TX
- R9: value R_Small -> RX
- TP13: value TestPoint -> TX
- TP14: value TestPoint -> RX
- TP15: value TestPoint -> RESET
- TP16: value TestPoint -> BOOT
Other:
- moved on the sheet: D11, D13, D7, R19, R8, R9

Commit message: polished up schematic
Parts:
- added TP12: SCL, symbol Connector:TestPoint
- added TP9: SDA, symbol Connector:TestPoint
- SW1: renamed from SW7; value SW_Push -> RESET
- SW2: renamed from SW8; value SW_Push -> BOOT
- renumbered C79 to C20, C80 to C21, C81 to C22, C82 to C23, C83 to C24, C84 to C25, C85 to C26, D7 to D10, J10 to J2, J9 to J3, R65 to R26, R66 to R27, R67 to R28, R8 to R29, R9 to R30, R68 to R31, R10 to R32, R19 to R33, R69 to R34, R70 to R35, R74 to R36, TP14 to TP10, TP16 to TP11, TP13 to TP7, TP15 to TP8, U16 to U5
Connections:
- net +3V3: now also TP12.1, TP9.1
Other:
- note added: "I2C Expansion"
- note removed: "I2C Expansion (light sensor?)"
- note removed: "creates RC delay on power up"
- company: (none) -> Jennifer Li
- title: (none) -> ESP32 S3 WROOM1 Microcontroller
- moved on the sheet: C20, D10, D11, J2, J3, R26, R27, R28, R29, R30, R36, SW1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
