File: Hardware/MCU.kicad_sch (KiCad schematic)
At the start: 33 parts, among them J2 Conn_01x04, J3 Conn_01x04, SW1 RESET, SW2 BOOT, U5 ESP32-S3-WROOM-1

Commit message: switch to macbook
Parts:
- removed D10: TX, symbol Device:LED_Small
- removed D11: RX, symbol Device:LED_Small
- removed R29: TX, symbol Device:R_Small
- removed R30: RX, symbol Device:R_Small
- C20: footprint (none) -> Capacitor_SMD:C_0603_1608Metric_Pad1.08x0.95mm_HandSolder; P/N (none) -> GXT188R71C105KE13D
- C21: footprint (none) -> Capacitor_SMD:C_0805_2012Metric_Pad1.18x1.45mm_HandSolder; P/N (none) -> MSAST21GBB5106MTNA01
- C22, C23, C24, C25, C26: footprint (none) -> Capacitor_SMD:C_0603_1608Metric_Pad1.08x0.95mm_HandSolder; P/N (none) -> GRM188R72A104KA35D
- D12, D13: footprint (none) -> LED_SMD:LED_0805_2012Metric_Pad1.15x1.40mm_HandSolder; P/N (none) -> LTST-C170TBKT
Other:
- moved on the sheet: D12, D13, R32, R33, TP10, TP11, TP7, TP8

Commit message: final touches to sch, switch out microphone
Parts:
- D12: value RESET -> RESET_LED
- D13: value BOOT -> BOOT_LED
- R26, R28: footprint (none) -> Resistor_SMD:R_0603_1608Metric_Pad0.98x0.95mm_HandSolder; P/N (none) -> ERJ-PC3B4701V
- R27, R31: footprint (none) -> Resistor_SMD:R_0201_0603Metric_Pad0.64x0.40mm_HandSolder; P/N (none) -> RC0201FR-0710KL
- R32: value RESET -> R
- R33: value BOOT -> R
- R34, R35: footprint (none) -> Resistor_SMD:R_0805_2012Metric_Pad1.20x1.40mm_HandSolder; P/N (none) -> ERJ-S06J220V
- R36: footprint (none) -> Resistor_SMD:R_0805_2012Metric_Pad1.20x1.40mm_HandSolder; P/N (none) -> RNAN0805BKE499R
- SW1: value RESET -> RESET_SW
- SW2: value BOOT -> BOOT_SW
- TP10, TP12, TP7, TP9: footprint (none) -> TestPoint:TestPoint_Keystone_5000-5004_Miniature
- TP11: value BOOT -> BOOT_TP; footprint (none) -> TestPoint:TestPoint_Keystone_5000-5004_Miniature
- TP8: value RESET -> RESET_TP; footprint (none) -> TestPoint:TestPoint_Keystone_5000-5004_Miniature
Changed lines of the file:
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@@
 			)
 		)
-		(property "Footprint" ""
+		(property "Footprint" "TestPoint:TestPoint_Keystone_5000-5004_Miniature"
 			(at 39.37 116.84 0)
 			(hide yes)
@@
 			)
 		)
-		(property "Value" "BOOT"
+		(property "Value" "BOOT_LED"
 			(at 70.104 123.444 90)
 			(show_name no)
@@
 			)
 		)
-		(property "Footprint" ""
+		(property "Footprint" "TestPoint:TestPoint_Keystone_5000-5004_Miniature"
 			(at 31.75 82.55 0)
 			(hide yes)
@@
 			)
 		)
-		(property "Value" "BOOT"
+		(property "Value" "R"
 			(at 70.104 116.84 0)
 			(show_name no)
@@
 			)
 		)
-		(property "Value" "RESET"
+		(property "Value" "RESET_SW"
 			(at 43.18 50.7999 90)
 			(show_name no)
@@
 			)
 		)
-		(property "Footprint" ""
+		(property "Footprint" "Resistor_SMD:R_0805_2012Metric_Pad1.20x1.40mm_HandSolder"
 			(at 163.83 40.64 0)
 			(hide yes)
@@
 			)
 		)
-		(property "P/N" ""
+		(property "P/N" "RNAN0805BKE499R"
 			(at 163.83 40.64 0)
 			(hide yes)
@@
 			)
 		)
-		(property "Value" "BOOT"
+		(property "Value" "BOOT_TP"
 			(at 36.83 123.6979 0)
 			(show_name no)
@@
 			)
 		)
-		(property "Footprint" ""
+		(property "Footprint" "TestPoint:TestPoint_Keystone_5000-5004_Miniature"
 			(at 39.37 125.73 0)
 			(hide yes)
@@
 			)
 		)
-		(property "Value" "RESET"
+		(property "Value" "R"
 			(at 52.832 116.84 0)
 			(show_name no)
@@
 			)
 		)
-		(property "Footprint" ""
+		(property "Footprint" "TestPoint:TestPoint_Keystone_5000-5004_Miniature"
 			(at 44.45 82.55 0)
 			(hide yes)
@@
 			)
 		)
-		(property "Value" "RESET"
+		(property "Value" "RESET_TP"
 			(at 24.13 123.6979 0)
 			(show_name no)
@@
 			)
 		)
-		(property "Footprint" ""
+		(property "Footprint" "TestPoint:TestPoint_Keystone_5000-5004_Miniature"
 			(at 26.67 125.73 0)
 			(hide yes)
@@
 			)
 		)
-		(property "Footprint" ""
+		(property "Footprint" "Resistor_SMD:R_0603_1608Metric_Pad0.98x0.95mm_HandSolder"
 			(at 44.45 81.28 0)
 			(hide yes)
@@
 			)
 		)
-		(property "P/N" ""
+		(property "P/N" "ERJ-PC3B4701V"
 			(at 44.45 81.28 0)
 			(hide yes)
@@
 			)
 		)
-		(property "Value" "RESET"
+		(property "Value" "RESET_LED"
 			(at 52.832 123.444 90)
 			(show_name no)
@@
 			)
 		)
-		(property "Footprint" ""
+		(property "Footprint" "Resistor_SMD:R_0805_2012Metric_Pad1.20x1.40mm_HandSolder"
 			(at 111.76 49.53 0)
 			(hide yes)
@@
 			)
 		)
-		(property "P/N" ""
+		(property "P/N" "ERJ-S06J220V"
 			(at 111.76 49.53 0)
 			(hide yes)
@@
 			)
 		)
-		(property "Footprint" ""
+		(property "Footprint" "Resistor_SMD:R_0201_0603Metric_Pad0.64x0.40mm_HandSolder"
 			(at 38.1 35.56 0)
 			(hide yes)
@@
 			)
 		)
-		(property "P/N" ""
+		(property "P/N" "RC0201FR-0710KL"
 			(at 38.1 35.56 0)
 			(hide yes)
@@
 			)
 		)
-		(property "Footprint" ""
+		(property "Footprint" "Resistor_SMD:R_0805_2012Metric_Pad1.20x1.40mm_HandSolder"
 			(at 111.76 52.07 0)
 			(hide yes)
@@
 			)
 		)
-		(property "P/N" ""
+		(property "P/N" "ERJ-S06J220V"
 			(at 111.76 52.07 0)
 			(hide yes)
@@
 			)
 		)
-		(property "Value" "BOOT"
+		(property "Value" "BOOT_SW"
 			(at 66.04 50.7999 90)
 			(show_name no)
@@
 			)
 		)
-		(property "Footprint" ""
+		(property "Footprint" "Resistor_SMD:R_0201_0603Metric_Pad0.64x0.40mm_HandSolder"
 			(at 64.77 39.37 0)
 			(hide yes)
@@
 			)
 		)
-		(property "P/N" ""
+		(property "P/N" "RC0201FR-0710KL"
 			(at 64.77 39.37 0)
 			(hide yes)
@@
 			)
 		)
-		(property "Footprint" ""
+		(property "Footprint" "Resistor_SMD:R_0603_1608Metric_Pad0.98x0.95mm_HandSolder"
 			(at 31.75 81.28 0)
 			(hide yes)
@@
 			)
 		)
-		(property "P/N" ""
+		(property "P/N" "ERJ-PC3B4701V"
 			(at 31.75 81.28 0)
 			(hide yes)
@@
 			)
 		)
-		(property "Footprint" ""
+		(property "Footprint" "TestPoint:TestPoint_Keystone_5000-5004_Miniature"
 			(at 26.67 116.84 0)
 			(hide yes)
