File: Hardware/PowerRegulation.kicad_sch (KiCad schematic)
At the start: 54 parts, among them Q4 AO3401A, U1 TPS56637RPAR, U14 AMS1117-3.3, U15 RT9193-33GB, U2 STUSB4500QTR

Commit message: switch to desktop
Parts:
- D1: value LED -> 9V
- D10: value LED -> PD_FAULT
- D2: value LED -> 5V
- D3: value LED -> 3V3
- D6: value LED -> 3V3_F
- TP3: value TestPoint -> 9V
- TP4: value TestPoint -> 5V
- TP5: value TestPoint -> 3V3
- TP6: value TestPoint -> 3V3_F
Other:
- note added: "Board requires initial PD controller programming through NVM Set POWER_ONLY_ABOVE_5V = 1 in NVM default I2C address: 0x28"
- note removed: "I2C for NVM programming"
- note removed: "Set POWER_ONLY_ABOVE_5V = 1 in NVM"
- note removed: "default I2C address: 0x28"
Changed lines of the file:
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@@
 	(text "place GND vias on exposed pad\n.3/.6 3x3"
 		(exclude_from_sim no)
-		(at 116.332 179.832 0)
+		(at 29.972 177.546 0)
 		(effects
 			(font
@@
 	(text "ensures gate voltage\ntracks source voltage"
 		(exclude_from_sim no)
-		(at 123.698 162.306 0)
+		(at 124.46 162.56 0)
 		(effects
 			(font
@@
 		)
 	)
-	(text "I2C for NVM programming"
-		(exclude_from_sim no)
-		(at 27.432 173.736 0)
-		(effects
-			(font
-				(size 1.27 1.27)
-			)
-			(justify left)
-		)
-	)
 	(text "Vout = 0.6 x (1 + Rfbt/Rfbb)\nVout = 0.6 x (1 + 73.2k/10k)\nVout = 0.6 x (1 + 7.32) = 4.992"
 		(exclude_from_sim no)
@@
 		)
 	)
+	(text "Board requires initial PD controller programming through NVM\nSet POWER_ONLY_ABOVE_5V = 1 in NVM\ndefault I2C address: 0x28"
+		(exclude_from_sim no)
+		(at 182.118 126.746 0)
+		(effects
+			(font
+				(size 1.778 1.778)
+			)
+			(justify left)
+		)
+	)
 	(text "CC1DB and CC2DB to CC1 and CC2\nfor dead-battery mode"
 		(exclude_from_sim no)
@@
 		)
 	)
-	(text "default I2C address: 0x28"
-		(exclude_from_sim no)
-		(at 27.432 171.196 0)
-		(effects
-			(font
-				(size 1.27 1.27)
-			)
-			(justify left)
-		)
-	)
 	(text "RESET active high"
 		(exclude_from_sim no)
@@
 		)
 	)
-	(text "Set POWER_ONLY_ABOVE_5V = 1 in NVM"
-		(exclude_from_sim no)
-		(at 57.15 179.324 0)
-		(effects
-			(font
-				(size 1.27 1.27)
-			)
-		)
-	)
 	(text "electrolytic\nbulk stability"
 		(exclude_from_sim no)
@@
 			)
 		)
-		(property "Value" "TestPoint"
+		(property "Value" "9V"
 			(at 207.01 94.7419 0)
 			(show_name no)
@@
 			)
 		)
-		(property "Value" "LED"
+		(property "Value" "3V3_F"
 			(at 262.89 51.1174 90)
 			(show_name no)
@@
 			)
 		)
-		(property "Value" "LED"
+		(property "Value" "PD_FAULT"
 			(at 208.28 51.1174 90)
 			(show_name no)
@@
 			)
 		)
-		(property "Value" "TestPoint"
+		(property "Value" "3V3"
 			(at 240.03 94.7419 0)
 			(show_name no)
@@
 			)
 		)
-		(property "Value" "LED"
+		(property "Value" "3V3"
 			(at 250.19 51.1174 90)
 			(show_name no)
@@
 			)
 		)
-		(property "Value" "LED"
+		(property "Value" "5V"
 			(at 236.22 51.1174 90)
 			(show_name no)
@@
 			)
 		)
-		(property "Value" "TestPoint"
+		(property "Value" "3V3_F"
 			(at 256.54 94.7419 0)
 			(show_name no)
@@
 			)
 		)
-		(property "Value" "TestPoint"
+		(property "Value" "5V"
 			(at 223.52 94.7419 0)
 			(show_name no)
@@
 			)
 		)
-		(property "Value" "LED"
+		(property "Value" "9V"
 			(at 222.25 51.1174 90)
 			(show_name no)

Commit message: polished up schematic
Parts:
- renumbered C47 to C10, C48 to C11, C6 to C12, C8 to C13, C76 to C14, C9 to C15, C77 to C16, C10 to C17, C78 to C18, C11 to C19, C3 to C2, C7 to C3, C73 to C4, C4 to C5, C5 to C6, C46 to C7, C74 to C8, C75 to C9, D10 to D5, D1 to D6, D2 to D7, D3 to D8, D6 to D9, Q4 to Q1, R77 to R10, R76 to R11, R63 to R12, R62 to R13, R1 to R14, R78 to R15, R57 to R16, R2 to R17, R58 to R18, R16 to R19, R17 to R20, R15 to R21, R4 to R22, R5 to R23, R6 to R24, R7 to R25, R61 to R5, R18 to R6, R64 to R7, R75 to R8, R59 to R9, U14 to U1, U1 to U2, U2 to U3, U15 to U4
Other:
- note added: "FCCM enabled"
- note added: "buck off during initial NVM programming"
- note added: "caps rated 2-3x input voltage"
- note removed: "Float MODE pin for FCCM mode, reduces noise"
- note removed: "caps rated ideally >30V"
- note removed: "chip off during initial NVM programming"
- note removed: "damp gate oscillation and slow turn on, prevent inrush current spike"
- company: (none) -> Jennifer Li
- title: (none) -> Power Regulation
- moved on the sheet: TP4, TP5, TP6
