File: Hardware/PowerRegulation.kicad_sch (KiCad schematic)
At the start: 54 parts, among them Q1 AO3401A, U1 AMS1117-3.3, U2 TPS56637RPAR, U3 STUSB4500QTR, U4 RT9193-33GB

Commit message: switch to macbook
Parts:
- C10, C11, C16: footprint (none) -> Capacitor_SMD:C_0603_1608Metric_Pad1.08x0.95mm_HandSolder; P/N (none) -> GXT188R71C105KE13D
- C14, C18, C4, C7, C9: footprint (none) -> Capacitor_SMD:C_0603_1608Metric_Pad1.08x0.95mm_HandSolder; P/N (none) -> GRM188R72A104KA35D
- C3, C8: footprint (none) -> Capacitor_SMD:C_0805_2012Metric_Pad1.18x1.45mm_HandSolder; P/N (none) -> MSAST21GBB5106MTNA01
- D5: footprint (none) -> LED_SMD:LED_0805_2012Metric_Pad1.15x1.40mm_HandSolder; P/N (none) -> LTST-C170KRKT
- D6, D7, D8, D9: footprint (none) -> LED_SMD:LED_0805_2012Metric_Pad1.15x1.40mm_HandSolder; P/N (none) -> LTST-C170GKT
- L1: footprint (none) -> LED Sign:7443340330; P/N XAL7070-332MEB -> 7443340330
- R14, R17: footprint (none) -> Resistor_SMD:R_0402_1005Metric_Pad0.72x0.64mm_HandSolder
- R19: footprint (none) -> Resistor_SMD:R_0805_2012Metric_Pad1.20x1.40mm_HandSolder
- R20: footprint (none) -> Resistor_SMD:R_0201_0603Metric_Pad0.64x0.40mm_HandSolder
Changed lines of the file:
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@@
 			)
 		)
-		(property "Footprint" ""
+		(property "Footprint" "LED Sign:7443340330"
 			(at 116.84 33.02 0)
 			(hide yes)
@@
 			)
 		)
-		(property "P/N" "XAL7070-332MEB"
+		(property "P/N" "7443340330"
 			(at 116.84 33.02 0)
 			(hide yes)
@@
 			)
 		)
-		(property "Footprint" ""
+		(property "Footprint" "Capacitor_SMD:C_0603_1608Metric_Pad1.08x0.95mm_HandSolder"
 			(at 147.32 92.71 0)
 			(hide yes)
@@
 			)
 		)
-		(property "P/N" ""
+		(property "P/N" "GRM188R72A104KA35D"
 			(at 147.32 92.71 0)
 			(hide yes)
@@
 			)
 		)
-		(property "Footprint" ""
+		(property "Footprint" "Capacitor_SMD:C_0805_2012Metric_Pad1.18x1.45mm_HandSolder"
 			(at 70.8152 92.71 0)
 			(hide yes)
@@
 			)
 		)
-		(property "P/N" ""
+		(property "P/N" "MSAST21GBB5106MTNA01"
 			(at 69.85 88.9 0)
 			(hide yes)
@@
 			)
 		)
-		(property "Footprint" ""
+		(property "Footprint" "Capacitor_SMD:C_0603_1608Metric_Pad1.08x0.95mm_HandSolder"
 			(at 45.72 88.9 0)
 			(hide yes)
@@
 			)
 		)
-		(property "P/N" ""
+		(property "P/N" "GRM188R72A104KA35D"
 			(at 45.72 88.9 0)
 			(hide yes)
@@
 			)
 		)
-		(property "Footprint" ""
+		(property "Footprint" "Capacitor_SMD:C_0603_1608Metric_Pad1.08x0.95mm_HandSolder"
 			(at 91.44 128.27 0)
 			(hide yes)
@@
 			)
 		)
-		(property "P/N" ""
+		(property "P/N" "GXT188R71C105KE13D"
 			(at 91.44 128.27 0)
 			(hide yes)
@@
 			)
 		)
-		(property "Footprint" ""
+		(property "Footprint" "LED_SMD:LED_0805_2012Metric_Pad1.15x1.40mm_HandSolder"
 			(at 259.08 48.26 0)
 			(hide yes)
@@
 			)
 		)
+		(property "P/N" "LTST-C170GKT"
+			(at 259.08 48.26 90)
+			(hide yes)
+			(show_name no)
+			(do_not_autoplace no)
+			(effects
+				(font
+					(size 1.27 1.27)
+				)
+			)
+		)
 		(pin "2"
 		)
@@
 			)
 		)
-		(property "Footprint" ""
+		(property "Footprint" "Capacitor_SMD:C_0603_1608Metric_Pad1.08x0.95mm_HandSolder"
 			(at 57.15 138.43 0)
 			(hide yes)
@@
 			)
 		)
-		(property "P/N" ""
+		(property "P/N" "GRM188R72A104KA35D"
 			(at 57.15 138.43 0)
 			(hide yes)
@@
 			)
 		)
-		(property "Footprint" ""
+		(property "Footprint" "LED_SMD:LED_0805_2012Metric_Pad1.15x1.40mm_HandSolder"
 			(at 204.47 48.26 0)
 			(hide yes)
@@
 			)
 		)
+		(property "P/N" "LTST-C170KRKT"
+			(at 204.47 48.26 90)
+			(hide yes)
+			(show_name no)
+			(do_not_autoplace no)
+			(effects
+				(font
+					(size 1.27 1.27)
+				)
+			)
+		)
 		(pin "2"
 		)
@@
 			)
 		)
-		(property "Footprint" ""
+		(property "Footprint" "Capacitor_SMD:C_0805_2012Metric_Pad1.18x1.45mm_HandSolder"
 			(at 40.3352 92.71 0)
 			(hide yes)
@@
 			)
 		)
-		(property "P/N" ""
+		(property "P/N" "MSAST21GBB5106MTNA01"
 			(at 39.37 88.9 0)
 			(hide yes)
@@
 			)
 		)
-		(property "Footprint" ""
+		(property "Footprint" "Resistor_SMD:R_0402_1005Metric_Pad0.72x0.64mm_HandSolder"
 			(at 133.35 41.148 90)
 			(hide yes)
@@
 			)
 		)
-		(property "Footprint" ""
+		(property "Footprint" "Resistor_SMD:R_0201_0603Metric_Pad0.64x0.40mm_HandSolder"
 			(at 141.478 55.88 90)
 			(hide yes)
@@
 			)
 		)
-		(property "Footprint" ""
+		(property "Footprint" "Capacitor_SMD:C_0603_1608Metric_Pad1.08x0.95mm_HandSolder"
 			(at 160.02 91.44 0)
 			(hide yes)
@@
 			)
 		)
-		(property "P/N" ""
+		(property "P/N" "GRM188R72A104KA35D"
 			(at 160.02 91.44 0)
 			(hide yes)
@@
 			)
 		)
-		(property "Footprint" ""
+		(property "Footprint" "Capacitor_SMD:C_0603_1608Metric_Pad1.08x0.95mm_HandSolder"
 			(at 154.6352 95.25 0)
 			(hide yes)
@@
 			)
 		)
-		(property "P/N" ""
+		(property "P/N" "GXT188R71C105KE13D"
 			(at 153.67 91.44 0)
 			(hide yes)
@@
 			)
 		)
-		(property "Footprint" ""
+		(property "Footprint" "LED_SMD:LED_0805_2012Metric_Pad1.15x1.40mm_HandSolder"
 			(at 246.38 48.26 0)
 			(hide yes)
@@
 			)
 		)
+		(property "P/N" "LTST-C170GKT"
+			(at 246.38 48.26 90)
+			(hide yes)
+			(show_name no)
+			(do_not_autoplace no)
+			(effects
+				(font
+					(size 1.27 1.27)
+				)
+			)
+		)
 		(pin "2"
 		)
@@
 			)
 		)
-		(property "Footprint" ""
+		(property "Footprint" "LED_SMD:LED_0805_2012Metric_Pad1.15x1.40mm_HandSolder"
 			(at 232.41 48.26 0)
 			(hide yes)
@@
 			)
 		)
+		(property "P/N" "LTST-C170GKT"
+			(at 232.41 48.26 90)
+			(hide yes)
+			(show_name no)
+			(do_not_autoplace no)
+			(effects
+				(font
+					(size 1.27 1.27)
+				)
+			)
+		)
 		(pin "2"
 		)
@@
 			)
 		)
-		(property "Footprint" ""
+		(property "Footprint" "Resistor_SMD:R_0805_2012Metric_Pad1.20x1.40mm_HandSolder"
 			(at 141.478 45.72 90)
 			(hide yes)
@@
 			)
 		)
-		(property "Footprint" ""
+		(property "Footprint" "Resistor_SMD:R_0402_1005Metric_Pad0.72x0.64mm_HandSolder"
 			(at 116.84 47.498 90)
 			(hide yes)
@@
 			)
 		)
-		(property "Footprint" ""
+		(property "Footprint" "LED_SMD:LED_0805_2012Metric_Pad1.15x1.40mm_HandSolder"
 			(at 218.44 48.26 0)
 			(hide yes)
@@
 			)
 		)
+		(property "P/N" "LTST-C170GKT"
+			(at 218.44 48.26 90)
+			(hide yes)
+			(show_name no)
+			(do_not_autoplace no)
+			(effects
+				(font
+					(size 1.27 1.27)
+				)
+			)
+		)
 		(pin "2"
 		)
@@
 			)
 		)
-		(property "Footprint" ""
+		(property "Footprint" "Capacitor_SMD:C_0603_1608Metric_Pad1.08x0.95mm_HandSolder"
 			(at 93.98 128.27 0)
 			(hide yes)
@@
 			)
 		)
-		(property "P/N" ""
+		(property "P/N" "GXT188R71C105KE13D"
 			(at 93.98 128.27 0)
 			(hide yes)
@@
 			)
 		)
-		(property "Footprint" ""
+		(property "Footprint" "Capacitor_SMD:C_0603_1608Metric_Pad1.08x0.95mm_HandSolder"
 			(at 76.2 88.9 0)
 			(hide yes)
@@
 			)
 		)
-		(property "P/N" ""
+		(property "P/N" "GRM188R72A104KA35D"
 			(at 76.2 88.9 0)
 			(hide yes)

Commit message: final touches to sch, switch out microphone
Parts:
- D6: value 9V -> 9V_LED
- D7: value 5V -> 5V_LED
- D8: value 3V3 -> 3V3_LED
- D9: value 3V3_F -> 3V3_F_LED
- R10, R11, R12, R13, R15, R16, R5, R6, R7, R8: footprint (none) -> Resistor_SMD:R_0402_1005Metric_Pad0.72x0.64mm_HandSolder
- R18: footprint (none) -> Resistor_SMD:R_0603_1608Metric_Pad0.98x0.95mm_HandSolder; P/N (none) -> ERA-3AEB223V
- R9: footprint (none) -> Resistor_SMD:R_0805_2012Metric_Pad1.20x1.40mm_HandSolder; P/N (none) -> RNAN0603BKE100R
- TP3: value 9V -> 9V_TP; footprint (none) -> TestPoint:TestPoint_Keystone_5000-5004_Miniature
- TP4: value 5V -> 5V_TP; footprint (none) -> TestPoint:TestPoint_Keystone_5000-5004_Miniature
- TP5: value 3V3 -> 3V3_TP; footprint (none) -> TestPoint:TestPoint_Keystone_5000-5004_Miniature
- TP6: value 3V3_F -> 3V3_F_TP; footprint (none) -> TestPoint:TestPoint_Keystone_5000-5004_Miniature
- U2: footprint RPA0010A -> LED Sign:TPS56637RPAR
- U4: footprint SOT-23-5_RIT -> LED Sign:RT9193-33
Changed lines of the file:
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@@
 			)
 		)
-		(property "Footprint" ""
+		(property "Footprint" "Resistor_SMD:R_0402_1005Metric_Pad0.72x0.64mm_HandSolder"
 			(at 63.5 157.988 90)
 			(hide yes)
@@
 			)
 		)
-		(property "Value" "9V"
+		(property "Value" "9V_TP"
 			(at 207.01 94.7419 0)
 			(show_name no)
@@
 			)
 		)
-		(property "Footprint" ""
+		(property "Footprint" "TestPoint:TestPoint_Keystone_5000-5004_Miniature"
 			(at 199.39 90.17 0)
 			(hide yes)
@@
 			)
 		)
-		(property "Footprint" ""
+		(property "Footprint" "Resistor_SMD:R_0402_1005Metric_Pad0.72x0.64mm_HandSolder"
 			(at 128.778 139.7 90)
 			(hide yes)
@@
 			)
 		)
-		(property "Footprint" ""
+		(property "Footprint" "Resistor_SMD:R_0402_1005Metric_Pad0.72x0.64mm_HandSolder"
 			(at 109.22 165.608 90)
 			(hide yes)
@@
 			)
 		)
-		(property "Footprint" ""
+		(property "Footprint" "Resistor_SMD:R_0402_1005Metric_Pad0.72x0.64mm_HandSolder"
 			(at 50.8 138.43 0)
 			(hide yes)
@@
 			)
 		)
-		(property "Footprint" "RPA0010A"
+		(property "Footprint" "LED Sign:TPS56637RPAR"
 			(at 85.09 45.72 0)
 			(hide yes)
@@
 			)
 		)
-		(property "Value" "3V3_F"
+		(property "Value" "3V3_F_LED"
 			(at 262.89 51.1174 90)
 			(show_name no)
@@
 			)
 		)
-		(property "Footprint" ""
+		(property "Footprint" "Resistor_SMD:R_0402_1005Metric_Pad0.72x0.64mm_HandSolder"
 			(at 63.5 164.592 90)
 			(hide yes)
@@
 			)
 		)
-		(property "Footprint" ""
+		(property "Footprint" "Resistor_SMD:R_0805_2012Metric_Pad1.20x1.40mm_HandSolder"
 			(at 105.41 156.21 0)
 			(hide yes)
@@
 			)
 		)
+		(property "P/N" "RNAN0603BKE100R"
+			(at 105.41 156.21 90)
+			(hide yes)
+			(show_name no)
+			(do_not_autoplace no)
+			(effects
+				(font
+					(size 1.27 1.27)
+				)
+			)
+		)
 		(pin "1"
 		)
@@
 			)
 		)
-		(property "Footprint" ""
+		(property "Footprint" "Resistor_SMD:R_0402_1005Metric_Pad0.72x0.64mm_HandSolder"
 			(at 118.618 139.7 90)
 			(hide yes)
@@
 			)
 		)
-		(property "Footprint" "SOT-23-5_RIT"
+		(property "Footprint" "LED Sign:RT9193-33"
 			(at 107.95 85.09 0)
 			(hide yes)
@@
 			)
 		)
-		(property "Footprint" ""
+		(property "Footprint" "Resistor_SMD:R_0402_1005Metric_Pad0.72x0.64mm_HandSolder"
 			(at 109.22 168.148 90)
 			(hide yes)
@@
 			)
 		)
-		(property "Footprint" ""
+		(property "Footprint" "Resistor_SMD:R_0402_1005Metric_Pad0.72x0.64mm_HandSolder"
 			(at 108.458 139.7 90)
 			(hide yes)
@@
 			)
 		)
-		(property "Value" "3V3"
+		(property "Value" "3V3_TP"
 			(at 242.57 94.7419 0)
 			(show_name no)
@@
 			)
 		)
-		(property "Footprint" ""
+		(property "Footprint" "TestPoint:TestPoint_Keystone_5000-5004_Miniature"
 			(at 234.95 90.17 0)
 			(hide yes)
@@
 			)
 		)
-		(property "Value" "3V3"
+		(property "Value" "3V3_LED"
 			(at 250.19 51.1174 90)
 			(show_name no)
@@
 			)
 		)
-		(property "Footprint" ""
+		(property "Footprint" "Resistor_SMD:R_0402_1005Metric_Pad0.72x0.64mm_HandSolder"
 			(at 63.5 38.1 0)
 			(hide yes)
@@
 			)
 		)
-		(property "Value" "5V"
+		(property "Value" "5V_LED"
 			(at 236.22 51.1174 90)
 			(show_name no)
@@
 			)
 		)
-		(property "Value" "3V3_F"
+		(property "Value" "3V3_F_TP"
 			(at 259.08 94.7419 0)
 			(show_name no)
@@
 			)
 		)
-		(property "Footprint" ""
+		(property "Footprint" "TestPoint:TestPoint_Keystone_5000-5004_Miniature"
 			(at 251.46 90.17 0)
 			(hide yes)
@@
 			)
 		)
-		(property "Value" "5V"
+		(property "Value" "5V_TP"
 			(at 224.79 94.7419 0)
 			(show_name no)
@@
 			)
 		)
-		(property "Footprint" ""
+		(property "Footprint" "TestPoint:TestPoint_Keystone_5000-5004_Miniature"
 			(at 217.17 90.17 0)
 			(hide yes)
@@
 			)
 		)
-		(property "Value" "9V"
+		(property "Value" "9V_LED"
 			(at 222.25 51.1174 90)
 			(show_name no)
@@
 			)
 		)
-		(property "Footprint" ""
+		(property "Footprint" "Resistor_SMD:R_0603_1608Metric_Pad0.98x0.95mm_HandSolder"
 			(at 134.62 151.892 90)
 			(hide yes)
@@
 			)
 		)
+		(property "P/N" "ERA-3AEB223V"
+			(at 134.62 153.67 0)
+			(hide yes)
+			(show_name no)
+			(do_not_autoplace no)
+			(effects
+				(font
+					(size 1.27 1.27)
+				)
+			)
+		)
 		(pin "1"
 		)
@@
 			)
 		)
-		(property "Footprint" ""
+		(property "Footprint" "Resistor_SMD:R_0402_1005Metric_Pad0.72x0.64mm_HandSolder"
 			(at 109.22 167.132 90)
 			(hide yes)
